Commit message: Add Kimchi description

File: andino_gz/urdf/include/kimchi_materials.xacro (robot description, xacro)
@@ -3,14 +3,4 @@
     <!-- Chassis -->
     <gazebo reference="base_link">
-      <visual>
-        <material>
-          <ambient>0.0 0.0 1.0 1.0</ambient>
-          <diffuse>0.0 0.0 1.0 1.0</diffuse>
-          <specular>0.1 0.1 0.1 1.0</specular>
-          <emissive>0.0 0.0 0.0 1.0</emissive>
-        </material>
-      </visual>
-    </gazebo>
-    <gazebo reference="second_base_link">
       <visual>
         <material>
@@ -43,6 +33,6 @@
       </visual>
     </gazebo>
-    <!-- Caster wheel -->
-    <gazebo reference="caster_rotation_link">
+    <!-- Caster wheels -->
+    <gazebo reference="left_caster_rotation_link">
       <visual>
         <material>
@@ -54,5 +44,5 @@
       </visual>
     </gazebo>
-    <gazebo reference="caster_base_link">
+    <gazebo reference="left_caster_base_link">
       <visual>
         <material>
@@ -64,5 +54,35 @@
       </visual>
     </gazebo>
-    <gazebo reference="caster_wheel_link">
+    <gazebo reference="left_caster_wheel_link">
+      <visual>
+        <material>
+          <ambient>0.1 0.1 0.1 1.0</ambient>
+          <diffuse>0.02 0.02 0.02 1.0</diffuse>
+          <specular>0.1 0.1 0.1 1.0</specular>
+          <emissive>0.0 0.0 0.0 1.0</emissive>
+        </material>
+      </visual>
+    </gazebo>
+    <gazebo reference="right_caster_rotation_link">
+      <visual>
+        <material>
+          <ambient>0.2 0.2 0.2 1.0</ambient>
+          <diffuse>0.3 0.3 0.3 1.0</diffuse>
+          <specular>0.9 0.9 0.9 1.0</specular>
+          <emissive>0.0 0.0 0.0 1.0</emissive>
+        </material>
+      </visual>
+    </gazebo>
+    <gazebo reference="right_caster_base_link">
+      <visual>
+        <material>
+          <ambient>0.2 0.2 0.2 1.0</ambient>
+          <diffuse>0.3 0.3 0.3 1.0</diffuse>
+          <specular>0.9 0.9 0.9 1.0</specular>
+          <emissive>0.0 0.0 0.0 1.0</emissive>
+        </material>
+      </visual>
+    </gazebo>
+    <gazebo reference="right_caster_wheel_link">
       <visual>
         <material>

File: andino_gz/urdf/kimchi_gz.urdf.xacro (robot description, xacro)
@@ -1,5 +1,5 @@
 <?xml version="1.0"?>
-<robot xmlns:xacro="http://www.ros.org/wiki/xacro" name="andino">
-  <xacro:include filename="$(find andino_description)/urdf/andino.urdf.xacro"/>
+<robot xmlns:xacro="http://www.ros.org/wiki/xacro" name="kimchi">
+  <xacro:include filename="$(find kimchi_description)/urdf/kimchi.urdf.xacro"/>
   <gazebo>
     <plugin
@@ -8,6 +8,6 @@
       <left_joint>left_wheel_joint</left_joint>
       <right_joint>right_wheel_joint</right_joint>
-      <wheel_separation>0.137</wheel_separation>
-      <wheel_radius>0.033</wheel_radius>
+      <wheel_separation>0.252</wheel_separation>
+      <wheel_radius>0.055</wheel_radius>
       <!--
       Odometry in the diff drive plugin is quite bad, therefore
@@ -38,6 +38,8 @@
       <joint_name>left_wheel_joint</joint_name>
       <joint_name>right_wheel_joint</joint_name>
-      <joint_name>caster_wheel_joint</joint_name>
-      <joint_name>caster_rotation_joint</joint_name>
+      <joint_name>left_caster_wheel_joint</joint_name>
+      <joint_name>left_caster_rotation_joint</joint_name>
+      <joint_name>right_caster_wheel_joint</joint_name>
+      <joint_name>right_caster_rotation_joint</joint_name>
     </plugin>
   </gazebo>
@@ -70,30 +72,4 @@
     </sensor>
   </gazebo>
-  <gazebo reference="camera_link">
-    <sensor name="camera" type="camera">
-      <gz_frame_id>camera_link</gz_frame_id>
-      <camera>
-        <horizontal_fov>1.047</horizontal_fov>
-        <image>
-          <width>640</width>
-          <height>480</height>
-        </image>
-        <clip>
-          <near>0.1</near>
-          <far>100</far>
-        </clip>
-        <distortion>
-          <k1>0.0</k1>
-          <k2>0.0</k2>
-          <k3>0.0</k3>
-          <p1>0.0</p1>
-          <p2>0.0</p2>
-        </distortion>
-      </camera>
-      <always_on>1</always_on>
-      <update_rate>30</update_rate>
-      <visualize>true</visualize>
-    </sensor>
-  </gazebo>
-  <xacro:include filename="$(find andino_gz)/urdf/include/andino_materials.xacro"/>
+  <xacro:include filename="$(find andino_gz)/urdf/include/kimchi_materials.xacro"/>
 </robot>
