Commit message: Add bumper and button to diffdrive

File: kimchi_description/urdf/include/common_sensors.urdf.xacro (robot description, xacro)
@@ -42,3 +42,24 @@
   </joint>
 </xacro:macro>
+<!-- Bumpers and button -->
+<xacro:macro name="digital_sensors" params="parent_link hardware_props">
+  <!-- Left Bumper -->
+  <link name="${hardware_props['left_bumper_name']}_link"/>
+  <joint name="${hardware_props['left_bumper_name']}" type="continuous">
+    <parent link="${parent_link}"/>
+    <child link="${hardware_props['left_bumper_name']}_link"/>
+  </joint>
+  <!-- Right Bumper -->
+  <link name="${hardware_props['right_bumper_name']}_link"/>
+  <joint name="${hardware_props['right_bumper_name']}" type="continuous">
+    <parent link="${parent_link}"/>
+    <child link="${hardware_props['right_bumper_name']}_link"/>
+  </joint>
+  <!-- Button -->
+  <link name="${hardware_props['button_name']}_link"/>
+  <joint name="${hardware_props['button_name']}" type="continuous">
+    <parent link="${parent_link}"/>
+    <child link="${hardware_props['button_name']}_link"/>
+  </joint>
+</xacro:macro>
 </robot>

File: kimchi_description/urdf/include/kimchi_control.urdf.xacro (robot description, xacro)
@@ -13,4 +13,7 @@
         <param name="left_wheel_name">${hardware_props['left_wheel_name']}</param>
         <param name="right_wheel_name">${hardware_props['right_wheel_name']}</param>
+        <param name="left_bumper_name">${hardware_props['left_bumper_name']}</param>
+        <param name="right_bumper_name">${hardware_props['right_bumper_name']}</param>
+        <param name="button_name">${hardware_props['button_name']}</param>
         <param name="serial_device">${hardware_props['serial_device']}</param>
         <param name="baud_rate">${hardware_props['baud_rate']}</param>
@@ -34,4 +37,14 @@
         <state_interface name="position"/>
       </joint>
+      <!-- Bumpers and button -->
+      <joint name="${hardware_props['left_bumper_name']}">
+        <state_interface name="position"/>
+      </joint>
+      <joint name="${hardware_props['right_bumper_name']}">
+        <state_interface name="position"/>
+      </joint>
+      <joint name="${hardware_props['button_name']}">
+        <state_interface name="position"/>
+      </joint>
     </ros2_control>
   </xacro:macro>

File: kimchi_description/urdf/kimchi.urdf.xacro (robot description, xacro)
@@ -51,4 +51,6 @@
     <xacro:include filename="$(find ${package_name})/urdf/include/kimchi_control.urdf.xacro" />
     <xacro:control hardware_props="${hardware_props}" />
+    <!-- Bumper and button -->
+    <xacro:digital_sensors parent_link="base_link" hardware_props="${hardware_props}" />
   </xacro:if>
 </robot>

Commit message: Adds bumper

File: kimchi_description/urdf/include/common_sensors.urdf.xacro (robot description, xacro)
@@ -45,18 +45,20 @@
 <xacro:macro name="digital_sensors" params="parent_link hardware_props">
   <!-- Left Bumper -->
-  <link name="${hardware_props['left_bumper_name']}_link"/>
-  <joint name="${hardware_props['left_bumper_name']}" type="continuous">
+  <link name="${hardware_props['bumpers']['left']['name']}_link"/>
+  <joint name="${hardware_props['bumpers']['left']['name']}" type="fixed">
     <parent link="${parent_link}"/>
-    <child link="${hardware_props['left_bumper_name']}_link"/>
+    <child link="${hardware_props['bumpers']['left']['name']}_link"/>
+    <origin xyz="${hardware_props['bumpers']['left']['dx']} ${hardware_props['bumpers']['left']['dy']} ${hardware_props['bumpers']['left']['dz']}" rpy="0 0 0"/>
   </joint>
   <!-- Right Bumper -->
-  <link name="${hardware_props['right_bumper_name']}_link"/>
-  <joint name="${hardware_props['right_bumper_name']}" type="continuous">
+  <link name="${hardware_props['bumpers']['right']['name']}_link"/>
+  <joint name="${hardware_props['bumpers']['right']['name']}" type="fixed">
     <parent link="${parent_link}"/>
-    <child link="${hardware_props['right_bumper_name']}_link"/>
+    <child link="${hardware_props['bumpers']['right']['name']}_link"/>
+    <origin xyz="${hardware_props['bumpers']['right']['dx']} ${hardware_props['bumpers']['right']['dy']} ${hardware_props['bumpers']['right']['dz']}" rpy="0 0 0"/>
   </joint>
   <!-- Button -->
   <link name="${hardware_props['button_name']}_link"/>
-  <joint name="${hardware_props['button_name']}" type="continuous">
+  <joint name="${hardware_props['button_name']}" type="fixed">
     <parent link="${parent_link}"/>
     <child link="${hardware_props['button_name']}_link"/>

File: kimchi_description/urdf/include/kimchi_control.urdf.xacro (robot description, xacro)
@@ -13,6 +13,6 @@
         <param name="left_wheel_name">${hardware_props['left_wheel_name']}</param>
         <param name="right_wheel_name">${hardware_props['right_wheel_name']}</param>
-        <param name="left_bumper_name">${hardware_props['left_bumper_name']}</param>
-        <param name="right_bumper_name">${hardware_props['right_bumper_name']}</param>
+        <param name="left_bumper_name">${hardware_props['bumpers']['left']['name']}</param>
+        <param name="right_bumper_name">${hardware_props['bumpers']['right']['name']}</param>
         <param name="button_name">${hardware_props['button_name']}</param>
         <param name="serial_device">${hardware_props['serial_device']}</param>
@@ -38,13 +38,13 @@
       </joint>
       <!-- Bumpers and button -->
-      <joint name="${hardware_props['left_bumper_name']}">
+      <gpio name="${hardware_props['bumpers']['left']['name']}">
         <state_interface name="position"/>
-      </joint>
-      <joint name="${hardware_props['right_bumper_name']}">
+      </gpio>
+      <gpio name="${hardware_props['bumpers']['right']['name']}">
         <state_interface name="position"/>
-      </joint>
-      <joint name="${hardware_props['button_name']}">
+      </gpio>
+      <gpio name="${hardware_props['button_name']}">
         <state_interface name="position"/>
-      </joint>
+      </gpio>
     </ros2_control>
   </xacro:macro>

File: kimchi_description/urdf/kimchi.urdf.xacro (robot description, xacro)
@@ -47,10 +47,10 @@
                    sensor_prop="${sensor_prop}">
   </xacro:laser>
+  <!-- Bumper and button -->
+  <xacro:digital_sensors parent_link="base_link" hardware_props="${hardware_props}" />
   <!-- ros2_control -->
   <xacro:if value="$(arg use_real_ros_control)">
     <xacro:include filename="$(find ${package_name})/urdf/include/kimchi_control.urdf.xacro" />
     <xacro:control hardware_props="${hardware_props}" />
-    <!-- Bumper and button -->
-    <xacro:digital_sensors parent_link="base_link" hardware_props="${hardware_props}" />
   </xacro:if>
 </robot>
